Commit message: update urdf

File: navigation2/nav2_bringup/urdf/Lite3.urdf (robot description, URDF)
Before this commit: robot MiniLiteV3, 20 links, 19 joints
Links:
- removed link Lidar
- added link base_link
- added link livox_frame, mass 0.01; visual cylinder length=0.06 radius=0.04
Joints:
- removed joint Lidar_Joint
- added joint base_to_torso: type fixed, parent base_link, child TORSO, origin xyz=0 0 0 rpy=0 0 0
- added joint livox_joint: type fixed, parent TORSO, child livox_frame, origin xyz=0.31 0 0.079
